File: ClaptrapKiCad/clapstar.sch (KiCad schematic (older format))
At the start: 14 parts

Commit message: Added: PCB Design sketch, Dane.txt
Parts:
- added C1: 1uF, Capacitor_THT:C_Disc_D4.7mm_W2.5mm_P5.00mm, symbol Device:C
- added D1: 1N4148, Diode_THT:D_DO-35_SOD27_P7.62mm_Horizontal, symbol Diode:1N4148
- added J1: Conn_01x02_Female, Connector_Wire:SolderWire-0.1sqmm_1x02_P3.6mm_D0.4mm_OD1mm_Relief, symbol Connector:Conn_01x02_Female
- added J2: Conn_01x02_Female, TerminalBlock:TerminalBlock_Altech_AK300-2_P5.00mm, symbol Connector:Conn_01x02_Female
- added K1: ADW11, Relay_THT:Relay_1P1T_NO_10x24x18.8mm_Panasonic_ADW11xxxxW_THT, symbol Relay:ADW11
- added OUT1: LED, LED_THT:LED_D3.0mm, symbol Device:LED
- added R5: 820, Resistor_THT:R_Axial_DIN0207_L6.3mm_D2.5mm_P10.16mm_Horizontal, symbol Device:R
- added U2: L78L05_TO92, Package_TO_SOT_THT:TO-92_Inline, symbol Regulator_Linear:L78L05_TO92
- C2: renamed from C?; value C -> 100 nF; footprint (none) -> Capacitor_THT:C_Disc_D3.0mm_W2.0mm_P2.50mm
- C3: footprint (none) -> Capacitor_THT:CP_Radial_D5.0mm_P2.50mm
- C4: footprint (none) -> Capacitor_THT:C_Disc_D4.7mm_W2.5mm_P5.00mm
- CLAP1: renamed from D?; footprint (none) -> LED_THT:LED_D3.0mm
- MIC1: renamed from MK?; footprint (none) -> Connector_Wire:SolderWire-0.1sqmm_1x02_P3.6mm_D0.4mm_OD1mm
- POT1: renamed from RV?; value R_POT -> 10k; footprint (none) -> Potentiometer_THT:Potentiometer_Vishay_T73YP_Vertical
- R1, R2, R3, R4: footprint (none) -> Resistor_THT:R_Axial_DIN0207_L6.3mm_D2.5mm_P10.16mm_Horizontal
- R6: renamed from R?; value R -> 1k; footprint (none) -> Resistor_THT:R_Axial_DIN0207_L6.3mm_D2.5mm_P10.16mm_Horizontal
- gave numbers to parts that had none: 3
Connections:
- net +5V: now also D1.1 (K), K1.1, R5.2, U2.1 (VO)
- net 0: now also T2.3 (E), C1.1, J1.1 (Pin_1), U2.2 (GND)
- net at U1.1 (~RESET~/PB5): now also R6.2
- net at U1.2 (PB3): no longer R6.2
- net at T2.1 (C): now also D1.2 (A), K1.6, OUT1.1 (K)
- new net: J2.1 (Pin_1), K1.3
- new net: J2.2 (Pin_2), K1.5
- new net: OUT1.2 (A), R5.1
- new net: C1.2, J1.2 (Pin_2), U2.3 (VI)
Other:
- moved on the sheet: R6, T2
